Commit message: sensors

File: car4_description/urdf/mobile_base.xacro (robot description, xacro)
@@ -7,5 +7,5 @@
     <xacro:property name="wheel_length" value="0.1" />
     <xacro:property name="column_radius" value="0.05" />
-    <xacro:property name="column_length" value="0.5" />
+    <xacro:property name="column_length" value="0.3" />
     <xacro:macro name="box_inertia" params="m l w h xyz rpy">
         <inertial>
@@ -23,5 +23,5 @@
             <inertia ixx="${(m/12)*(3*r*r + l*l)}" ixy="0.0" ixz="0.0"
                      iyy="${(m/12)*(3*r*r + l*l)}" iyz="0.0"
-                     izz="${(m*r*r)/2}"/>
+                     izz="${(m/2)*(r*r)}"/>
         </inertial>
     </xacro:macro>
@@ -32,5 +32,5 @@
             <inertia ixx="${(m/12)*(3*r*r + l*l)}" ixy="0.0" ixz="0.0"
                      iyy="${(m/12)*(3*r*r + l*l)}" iyz="0.0"
-                     izz="${(m*r*r)/2}"/>
+                     izz="${(m/2)*(r*r)}"/>
         </inertial>
     </xacro:macro>
@@ -43,4 +43,10 @@
     <material name="black">
         <color rgba="0.0 0.0 0.0 1" />
+    </material>
+    <material name="red">
+        <color rgba="1.0 0.0 0.0 1" />
+    </material>
+     <material name="green">
+        <color rgba="0.0 1.0 0.0 1" />
     </material>
     <link name="base_footprint" />
@@ -72,5 +78,5 @@
                 <cylinder radius="${column_radius}" length="${column_length}"/>
             </geometry>
-            <origin xyz="0 0 0.25" rpy="0 0 0" />
+            <origin xyz="0 0 0.15" rpy="0 0 0" />
             <material name="grey" />
         </visual>
@@ -79,8 +85,8 @@
                 <cylinder radius="${column_radius}" length="${column_length}"/>
             </geometry>
-            <origin xyz="0 0 0.25" rpy="0 0 0" />
+            <origin xyz="0 0 0.15" rpy="0 0 0" />
         </collision>
-        <xacro:wheel_inertia m="1.0" r="${column_radius}" l="${column_length}"
-                            xyz="0 0 0.25"  rpy="0.0 0.0 0.0" />
+        <xacro:wheel_inertia m="0.3" r="${column_radius}" l="${column_length}"
+                            xyz="0 0 0.15"  rpy="0.0 0.0 0.0" />
     </link>
     <joint name="base_second_joint" type="fixed">
@@ -138,5 +144,5 @@
         <visual>
             <geometry>
-                <cylinder radius="0.15" length="0.1"/>
+                <cylinder radius="${wheel_radius}" length="${wheel_length}"/>
             </geometry>
             <origin xyz="0.0 0.0 0.0" rpy="1.57 0.0 0.0"/>
@@ -161,5 +167,5 @@
         <visual>
             <geometry>
-                <cylinder radius="0.15" length="0.1"/>
+                <cylinder radius="${wheel_radius}" length="${wheel_length}"/>
             </geometry>
             <origin xyz="0.0 0.0 0.0" rpy="1.57 0.0 0.0"/>

File: car4_description/urdf/mobile_base_gazebo.xacro (robot description, xacro)
@@ -1,18 +1,29 @@
 <?xml version="1.0"?>
 <robot name="car4" xmlns:xacro="http://www.ros.org/wiki/xacro">
+      <!-- Zmienne definiujące współczynniki tarcia -->
+    <xacro:property name="mu1_value" value="0.1" />
+    <xacro:property name="mu2_value" value="0.1" />
     <gazebo reference="base_link">
         <material>Gazebo/Orange</material>
     </gazebo>
-    <gazebo reference="back_right_wheel_link">
+    <gazebo reference="rear_right_wheel_link">
         <material>Gazebo/Black</material>
+        <mu1>${mu1_value}</mu1>
+        <mu2>${mu2_value}</mu2>
     </gazebo>
-    <gazebo reference="back_left_wheel_link">
+    <gazebo reference="rear_left_wheel_link">
         <material>Gazebo/Black</material>
+        <mu1>${mu1_value}</mu1>
+        <mu2>${mu2_value}</mu2>
     </gazebo>
     <gazebo reference="front_right_wheel_link">
         <material>Gazebo/Black</material>
+        <mu1>${mu1_value}</mu1>
+        <mu2>${mu2_value}</mu2>
     </gazebo>
     <gazebo reference="front_left_wheel_link">
         <material>Gazebo/Black</material>
+        <mu1>${mu1_value}</mu1>
+        <mu2>${mu2_value}</mu2>
     </gazebo>
     <gazebo reference="second_link">
@@ -25,9 +36,11 @@
             <!-- Przypisanie przegubów kół (napędzanych) -->
             <left_joint>base_front_left_wheel_joint</left_joint>
+            <right_joint>base_front_right_wheel_joint</right_joint>
             <left_joint>base_rear_left_wheel_joint</left_joint>
-            <right_joint>base_front_right_wheel_joint</right_joint>
             <right_joint>base_rear_right_wheel_joint</right_joint>
             <!-- Parametry kół -->
             <wheel_separation>0.6</wheel_separation>
+            <wheel_separation>0.6</wheel_separation>
+            <wheel_diameter>0.3</wheel_diameter>
             <wheel_diameter>0.3</wheel_diameter>
             <!-- Topic do odbierania komend -->

File: car4_description/urdf/my_robot.urdf.xacro (robot description, xacro)
@@ -3,3 +3,6 @@
     <xacro:include filename="mobile_base.xacro" />
     <xacro:include filename="mobile_base_gazebo.xacro" />
+    <xacro:include filename="lidar.xacro" />
+    <xacro:include filename="imu.xacro" />
+    <xacro:include filename="gps.xacro" />
 </robot>
