Commit message: fiz nav

File: car4_description/urdf/lidar_laser.xacro (robot description, xacro)
@@ -24,15 +24,15 @@
         <child link="lidar_link"/>
     </joint>
-    <gazebo reference="lidar_link">
-        <sensor type="ray" name="lidar_sensor">
-            <update_rate>10.0</update_rate>
+   <gazebo reference="lidar_link">
+        <material>Gazebo/Red</material>
+        <sensor name="laser" type="ray">
+            <pose> 0 0 0 0 0 0 </pose>
             <visualize>true</visualize>
-            <!-- <topic>lidar_scan</topic>
-            <frame_name>lidar_link</frame_name> -->
+            <update_rate>60</update_rate>
             <ray>
                 <scan>
                     <horizontal>
-                        <samples>720</samples>
-                        <resolution>1</resolution>
+                        <samples>360</samples>
+                        <resolution>0.5</resolution>
                         <min_angle>-3.14</min_angle>
                         <max_angle>3.14</max_angle>
@@ -40,15 +40,15 @@
                 </scan>
                 <range>
-                    <min>0.1</min>
-                    <max>30.0</max>
+                    <min>0.3</min>
+                    <max>12</max>
+                    <resolution>0.01</resolution>
                 </range>
-                <noise>
-                    <type>gaussian</type>
-                    <mean>0.5</mean>
-                    <stddev>0.01</stddev>
-                </noise>
             </ray>
-            <plugin name="lidar" filename="libgazebo_ros_ray_sensor.so">
-             <outputType>laser</outputType>
+            <plugin name="laser_controller" filename="libgazebo_ros_ray_sensor.so">
+                <ros>
+                    <argument>~/out:=scan</argument>
+                </ros>
+                <output_type>sensor_msgs/LaserScan</output_type>
+                <frame_name>lidar_link</frame_name>
             </plugin>
         </sensor>

File: car4_description/urdf/mobile_base.xacro (robot description, xacro)
@@ -65,5 +65,5 @@
             <origin xyz="0 0 0.1" rpy="0 0 0"/>
         </collision>
-        <xacro:box_inertia m="5.0" l="${base_length}" w="${base_width}" h="${base_height}"
+        <xacro:box_inertia m="2.0" l="${base_length}" w="${base_width}" h="${base_height}"
                             xyz="0 0 0.1"  rpy="0 0 0" />
     </link>
@@ -109,5 +109,5 @@
             <origin xyz="0.0 0.0 0.0" rpy="1.57 0.0 0.0"/>
         </collision>
-        <xacro:wheel_inertia m="1.0" r="${wheel_radius}" l="${wheel_length}"
+        <xacro:wheel_inertia m="0.3" r="${wheel_radius}" l="${wheel_length}"
                             xyz="0.0 0.0 0.0"  rpy="1.57 0.0 0.0" />
     </link>
@@ -132,5 +132,5 @@
             <origin xyz="0.0 0.0 0.0" rpy="1.57 0.0 0.0"/>
         </collision>
-        <xacro:wheel_inertia m="1.0" r="${wheel_radius}" l="${wheel_length}"
+        <xacro:wheel_inertia m="0.3" r="${wheel_radius}" l="${wheel_length}"
                             xyz="0.0 0.0 0.0"  rpy="1.57 0.0 0.0" />
     </link>
@@ -155,5 +155,5 @@
             <origin xyz="0.0 0.0 0.0" rpy="1.57 0.0 0.0"/>
         </collision>
-        <xacro:wheel_inertia m="1.0" r="${wheel_radius}" l="${wheel_length}"
+        <xacro:wheel_inertia m="0.3" r="${wheel_radius}" l="${wheel_length}"
                             xyz="0.0 0.0 0.0"  rpy="1.57 0.0 0.0" />
     </link>
@@ -178,5 +178,5 @@
             <origin xyz="0.0 0.0 0.0" rpy="1.57 0.0 0.0"/>
         </collision>
-        <xacro:wheel_inertia m="1.0" r="${wheel_radius}" l="${wheel_length}"
+        <xacro:wheel_inertia m="0.3" r="${wheel_radius}" l="${wheel_length}"
                             xyz="0.0 0.0 0.0"  rpy="1.57 0.0 0.0" />
     </link>

File: car4_description/urdf/mobile_base_gazebo.xacro (robot description, xacro)
@@ -53,5 +53,5 @@
             <publish_steerangle>true</publish_steerangle>
             <!-- Ramki odometryczne -->
-            <odometry_frame>odom_demo</odometry_frame>
+            <odometry_frame>odom</odometry_frame>
             <robot_base_frame>base_footprint</robot_base_frame>
         </plugin>

File: car4_description/urdf/my_robot.urdf.xacro (robot description, xacro)
@@ -3,5 +3,5 @@
     <xacro:include filename="mobile_base.xacro" />
     <xacro:include filename="mobile_base_gazebo.xacro" />
-    <xacro:include filename="lidar.xacro" />
+    <xacro:include filename="lidar_laser.xacro" />
     <xacro:include filename="imu.xacro" />
     <xacro:include filename="gps.xacro" />
